File: eva-terminals.kicad_pcb (KiCad board)
At the start: 2 copper layers, 64 x 64 mm, 33 parts, among them J1 691403900006B, J2 691403900006B, J3 Conn_01x04, J4 691403900006B, J5 HEATER, J6 Conn_02x10_Odd_Even, J7 Conn_02x10_Odd_Even, J8 SPI, U1 LD39015M33R, U2 ADXL345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

Commit message: small changes
Other:
- board text added: "JLCJLCJLCJLC"
Changed lines of the file:
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@@
       (outputformat 1)
       (mirror false)
-      (drillshape 1)
+      (drillshape 0)
       (scaleselection 1)
-      (outputdirectory "")
+      (outputdirectory "gerbers/")
     )
   )
@@
     (fp_line (start -1.6 0.8) (end -1.6 -0.8) (layer "F.Fab") (width 0.1))
     (fp_line (start 1.6 0.8) (end -1.6 0.8) (layer "F.Fab") (width 0.1))
-    (pad "1" smd roundrect locked (at -1.4625 0 90) (size 1.125 1.75) (layers "F.Cu" "F.Paste" "F.Mask") (roundrect_rratio 0.222222)
+    (pad "1" smd roundrect locked (at -1.4625 0 90) (size 1.125 1.75) (layers "F.Cu" "F.Paste" "F.Mask") (roundrect_rratio 0.2222222222)
       (net 34 "CHAMBER_TEMP") (pintype "passive"))
-    (pad "2" smd roundrect locked (at 1.4625 0 90) (size 1.125 1.75) (layers "F.Cu" "F.Paste" "F.Mask") (roundrect_rratio 0.222222)
+    (pad "2" smd roundrect locked (at 1.4625 0 90) (size 1.125 1.75) (layers "F.Cu" "F.Paste" "F.Mask") (roundrect_rratio 0.2222222222)
       (net 32 "GNDREF") (pintype "passive"))
     (model "${KICAD6_3DMODEL_DIR}/Resistor_SMD.3dshapes/R_1206_3216Metric.wrl"
@@
     (fp_line (start -2.45 9.2) (end -2.45 -2.3) (layer "F.Fab") (width 0.1))
     (fp_line (start 8.75 -2.3) (end 8.75 2.2) (layer "F.Fab") (width 0.1))
-    (pad "1" thru_hole roundrect locked (at 0 0 180) (size 1.7 1.95) (drill 0.95) (layers *.Cu *.Mask) (roundrect_rratio 0.147059)
+    (pad "1" thru_hole roundrect locked (at 0 0 180) (size 1.7 1.95) (drill 0.95) (layers *.Cu *.Mask) (roundrect_rratio 0.1470588235)
       (net 8 "EXTRUDER_1") (pinfunction "Pin_1") (pintype "passive"))
     (pad "2" thru_hole oval locked (at 2.5 0 180) (size 1.7 1.95) (drill 0.95) (layers *.Cu *.Mask)
@@
     (effects (font (size 0.8 0.8) (thickness 0.15)))
   )
+  (gr_text "JLCJLCJLCJLC" (at 94 120) (layer "F.SilkS")
+    (effects (font (size 0.8 0.8) (thickness 0.15)))
+  )
