File: eva-terminals.kicad_sch (KiCad schematic)
At the start: 29 parts, among them J1 691403900006B, J2 691403900006B, J3 Conn_01x04, J4 691403900006B, J5 HEATER, J6 Conn_02x10_Odd_Even, J7 Conn_02x10_Odd_Even, J8 SPI, U1 LD39015M33R, U2 ADXL345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

Commit message: small changes
Parts:
- added JP5: SolderJumper_2_Open, Jumper:SolderJumper-2_P1.3mm_Open_RoundedPad1.0x1.5mm, symbol Jumper:SolderJumper_2_Open
Connections:
- net GND: now also J1.5 (Pin_5), J1.A5 (Pin_A5); no longer J1.6 (Pin_6), J1.A6 (Pin_A6)
- net HEATER_PWR: now also JP5.2 (B)
- net PROBE: now also J1.6 (Pin_6), J1.A6 (Pin_A6); no longer J1.4 (Pin_4), J1.A4 (Pin_A4)
- net PROBE_PWR: now also J1.4 (Pin_4), J1.A4 (Pin_A4), JP5.1 (A); no longer J1.5 (Pin_5), J1.A5 (Pin_A5)
Changed lines of the file:
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@@
   (junction (at 43.18 35.56) (diameter 0) (color 0 0 0 0)
+  )
+  (junction (at 96.52 87.63) (diameter 0) (color 0 0 0 0)
   )
   (junction (at 22.225 94.615) (diameter 0) (color 0 0 0 0)
@@
     (stroke (width 0) (type default) (color 0 0 0 0))
   )
+  (wire (pts (xy 96.52 87.63) (xy 96.52 81.28))
+    (stroke (width 0) (type default) (color 0 0 0 0))
+  )
   (polyline (pts (xy 88.9 152.4) (xy 88.9 190.5))
     (stroke (width 0) (type default) (color 0 0 0 0))
@@
     (stroke (width 0) (type default) (color 0 0 0 0))
   )
+  (wire (pts (xy 226.06 78.74) (xy 229.87 78.74))
+    (stroke (width 0) (type default) (color 0 0 0 0))
+  )
   (wire (pts (xy 51.435 118.745) (xy 51.435 120.65))
     (stroke (width 0) (type default) (color 0 0 0 0))
@@
     (stroke (width 0) (type default) (color 0 0 0 0))
   )
+  (wire (pts (xy 106.68 81.28) (xy 111.76 81.28))
+    (stroke (width 0) (type default) (color 0 0 0 0))
+  )
   (wire (pts (xy 22.225 106.045) (xy 22.225 108.585))
     (stroke (width 0) (type default) (color 0 0 0 0))
@@
     (stroke (width 0) (type default) (color 0 0 0 0))
   )
-  (wire (pts (xy 226.695 81.28) (xy 229.87 81.28))
-    (stroke (width 0) (type default) (color 0 0 0 0))
-  )
   (wire (pts (xy 43.18 55.88) (xy 43.18 60.96))
     (stroke (width 0) (type default) (color 0 0 0 0))
@@
   )
   (wire (pts (xy 81.28 93.98) (xy 86.36 93.98))
+    (stroke (width 0) (type default) (color 0 0 0 0))
+  )
+  (wire (pts (xy 224.79 81.28) (xy 229.87 81.28))
+    (stroke (width 0) (type default) (color 0 0 0 0))
+  )
+  (wire (pts (xy 96.52 81.28) (xy 99.06 81.28))
     (stroke (width 0) (type default) (color 0 0 0 0))
   )
@@
     )
   )
-  (global_label "PROBE_PWR" (shape input) (at 229.87 78.74 180) (fields_autoplaced)
-    (effects (font (size 1.27 1.27)) (justify right))
-    (property "Intersheet References" "${INTERSHEET_REFS}" (id 0) (at 216.2972 78.6606 0)
+  (global_label "PROBE_PWR" (shape input) (at 229.87 76.2 180) (fields_autoplaced)
+    (effects (font (size 1.27 1.27)) (justify right))
+    (property "Intersheet References" "${INTERSHEET_REFS}" (id 0) (at 216.2972 76.1206 0)
       (effects (font (size 1.27 1.27)) (justify right) hide)
     )
@@
     )
   )
-  (global_label "PROBE" (shape input) (at 229.87 76.2 180) (fields_autoplaced)
-    (effects (font (size 1.27 1.27)) (justify right))
-    (property "Intersheet References" "${INTERSHEET_REFS}" (id 0) (at 221.2563 76.1206 0)
+  (global_label "PROBE" (shape input) (at 224.79 81.28 180) (fields_autoplaced)
+    (effects (font (size 1.27 1.27)) (justify right))
+    (property "Intersheet References" "${INTERSHEET_REFS}" (id 0) (at 216.1763 81.2006 0)
       (effects (font (size 1.27 1.27)) (justify right) hide)
     )
@@
     (effects (font (size 1.27 1.27)) (justify left))
     (property "Intersheet References" "${INTERSHEET_REFS}" (id 0) (at 180.6685 67.2306 0)
+      (effects (font (size 1.27 1.27)) (justify left) hide)
+    )
+  )
+  (global_label "HEATER_PWR" (shape input) (at 111.76 81.28 0) (fields_autoplaced)
+    (effects (font (size 1.27 1.27)) (justify left))
+    (property "Intersheet References" "${INTERSHEET_REFS}" (id 0) (at 125.998 81.2006 0)
       (effects (font (size 1.27 1.27)) (justify left) hide)
     )
@@
     (pin "1")
   )
-  (symbol (lib_id "power:GND") (at 226.695 81.28 270) (mirror x) (unit 1)
-    (in_bom yes) (on_board yes)
-    (property "Reference" "#PWR0119" (id 0) (at 220.345 81.28 0)
-      (effects (font (size 1.27 1.27)) hide)
-    )
-    (property "Value" "GND" (id 1) (at 219.075 81.28 90)
-      (effects (font (size 1.27 1.27)) (justify left))
-    )
-    (property "Footprint" "" (id 2) (at 226.695 81.28 0)
-      (effects (font (size 1.27 1.27)) hide)
-    )
-    (property "Datasheet" "" (id 3) (at 226.695 81.28 0)
+  (symbol (lib_id "Jumper:SolderJumper_2_Open") (at 102.87 81.28 0) (unit 1)
+    (in_bom yes) (on_board yes) (fields_autoplaced)
+    (property "Reference" "JP5" (id 0) (at 102.87 76.4245 0))
+    (property "Value" "SolderJumper_2_Open" (id 1) (at 102.87 79.1996 0))
+    (property "Footprint" "Jumper:SolderJumper-2_P1.3mm_Open_RoundedPad1.0x1.5mm" (id 2) (at 102.87 81.28 0)
+      (effects (font (size 1.27 1.27)) hide)
+    )
+    (property "Datasheet" "~" (id 3) (at 102.87 81.28 0)
+      (effects (font (size 1.27 1.27)) hide)
+    )
+    (pin "1")
+    (pin "2")
+  )
+  (symbol (lib_id "power:GND") (at 226.06 78.74 270) (mirror x) (unit 1)
+    (in_bom yes) (on_board yes)
+    (property "Reference" "#PWR0119" (id 0) (at 219.71 78.74 0)
+      (effects (font (size 1.27 1.27)) hide)
+    )
+    (property "Value" "GND" (id 1) (at 218.44 78.74 90)
+      (effects (font (size 1.27 1.27)) (justify left))
+    )
+    (property "Footprint" "" (id 2) (at 226.06 78.74 0)
+      (effects (font (size 1.27 1.27)) hide)
+    )
+    (property "Datasheet" "" (id 3) (at 226.06 78.74 0)
       (effects (font (size 1.27 1.27)) hide)
     )
@@
       (reference "JP4") (unit 1) (value "SolderJumper_2_Open") (footprint "Jumper:SolderJumper-2_P1.3mm_Open_RoundedPad1.0x1.5mm")
     )
+    (path "/70852beb-7102-4701-922b-9248dc6321b9"
+      (reference "JP5") (unit 1) (value "SolderJumper_2_Open") (footprint "Jumper:SolderJumper-2_P1.3mm_Open_RoundedPad1.0x1.5mm")
+    )
     (path "/62e37993-d7e3-4eca-807c-0cee17f598bc"
